File: Electrical Design/pcb_tile_game.kicad_sch (KiCad schematic)
At the start: 40 parts, among them J1 Conn_01x05_Pin, J2 Conn_01x05_Socket, J3 Conn_01x05_Pin, J4 Conn_01x05_Socket, J5 Conn_01x05_Pin, J6 Conn_01x05_Socket, U2 ATtiny3217-M

Commit message: updated 3D models and silkscreen
Added magnetic connector models, LED models, changed path thickness, added title, revision, and logo to silkscreen.
Other:
- title: PCB Tile Game -> (none)
Changed lines of the file:
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@@
 	(generator_version "8.0")
 	(paper "A4")
-	(title_block
-		(title "PCB Tile Game")
-		(rev "0.1")
-	)
 	(junction
 		(at 124.46 104.14)
@@
 	(label "SPARE_5"
 		(at 21.59 71.12 0)
+		(fields_autoplaced yes)
 		(effects
 			(font
@@
 	(label "SIDE_4"
 		(at 74.93 58.42 180)
+		(fields_autoplaced yes)
 		(effects
 			(font
@@
 	(label "SPARE_1"
 		(at 74.93 50.8 180)
+		(fields_autoplaced yes)
 		(effects
 			(font
@@
 	(label "UPDI"
 		(at 74.93 35.56 180)
+		(fields_autoplaced yes)
 		(effects
 			(font
@@
 	(label "SPARE_6b"
 		(at 74.93 40.64 180)
+		(fields_autoplaced yes)
 		(effects
 			(font
@@
 	(label "SIDE_5"
 		(at 220.98 34.29 0)
+		(fields_autoplaced yes)
 		(effects
 			(font
@@
 	(label "SPARE_6a"
 		(at 74.93 38.1 180)
+		(fields_autoplaced yes)
 		(effects
 			(font
@@
 	(label "SIDE_5"
 		(at 74.93 43.18 180)
+		(fields_autoplaced yes)
 		(effects
 			(font
@@
 	(label "SPARE_6b"
 		(at 220.98 60.96 0)
+		(fields_autoplaced yes)
 		(effects
 			(font
@@
 	(label "SIDE_1"
 		(at 74.93 48.26 180)
+		(fields_autoplaced yes)
 		(effects
 			(font
@@
 	(label "LED"
 		(at 74.93 53.34 180)
+		(fields_autoplaced yes)
 		(effects
 			(font
@@
 	(label "SIDE_2"
 		(at 74.93 63.5 180)
+		(fields_autoplaced yes)
 		(effects
 			(font
@@
 	(label "UPDI"
 		(at 88.9 41.91 180)
+		(fields_autoplaced yes)
 		(effects
 			(font
@@
 	(label "SIDE_3"
 		(at 180.34 34.29 0)
+		(fields_autoplaced yes)
 		(effects
 			(font
@@
 	(label "SIDE_4"
 		(at 180.34 58.42 0)
+		(fields_autoplaced yes)
 		(effects
 			(font
@@
 	(label "SPARE_4b"
 		(at 21.59 68.58 0)
+		(fields_autoplaced yes)
 		(effects
 			(font
@@
 	(label "SIDE_1"
 		(at 140.97 34.29 0)
+		(fields_autoplaced yes)
 		(effects
 			(font
@@
 	(label "UPDI"
 		(at 140.97 31.75 0)
+		(fields_autoplaced yes)
 		(effects
 			(font
@@
 	(label "LED_OUT_1"
 		(at 281.94 111.76 180)
+		(fields_autoplaced yes)
 		(effects
 			(font
@@
 	(label "SPARE_2b"
 		(at 140.97 60.96 0)
+		(fields_autoplaced yes)
 		(effects
 			(font
@@
 	(label "LED"
 		(at 24.13 111.76 0)
+		(fields_autoplaced yes)
 		(effects
 			(font
@@
 	(label "SIDE_2"
 		(at 140.97 58.42 0)
+		(fields_autoplaced yes)
 		(effects
 			(font
@@
 	(label "SPARE_4b"
 		(at 180.34 60.96 0)
+		(fields_autoplaced yes)
 		(effects
 			(font
@@
 	(label "SIDE_6"
 		(at 220.98 58.42 0)
+		(fields_autoplaced yes)
 		(effects
 			(font
@@
 	(label "SPARE_2b"
 		(at 74.93 73.66 180)
+		(fields_autoplaced yes)
 		(effects
 			(font
@@
 	(label "SPARE_1"
 		(at 140.97 36.83 0)
+		(fields_autoplaced yes)
 		(effects
 			(font
@@
 	(label "SPARE_4a"
 		(at 180.34 55.88 0)
+		(fields_autoplaced yes)
 		(effects
 			(font
@@
 	(label "UPDI"
 		(at 180.34 31.75 0)
+		(fields_autoplaced yes)
 		(effects
 			(font
@@
 	(label "SPARE_3"
 		(at 180.34 36.83 0)
+		(fields_autoplaced yes)
 		(effects
 			(font
@@
 	(label "SPARE_2a"
 		(at 140.97 55.88 0)
+		(fields_autoplaced yes)
 		(effects
 			(font
@@
 	(label "SPARE_2a"
 		(at 74.93 76.2 180)
+		(fields_autoplaced yes)
 		(effects
 			(font
@@
 	(label "LED_OUT_1"
 		(at 33.02 142.24 180)
+		(fields_autoplaced yes)
 		(effects
 			(font
@@
 	(label "SPARE_6a"
 		(at 220.98 55.88 0)
+		(fields_autoplaced yes)
 		(effects
 			(font
@@
 	(label "SPARE_3"
 		(at 21.59 63.5 0)
+		(fields_autoplaced yes)
 		(effects
 			(font
@@
 	(label "UPDI"
 		(at 100.33 34.29 0)
+		(fields_autoplaced yes)
 		(effects
 			(font
@@
 	(label "UPDI"
 		(at 220.98 31.75 0)
+		(fields_autoplaced yes)
 		(effects
 			(font
@@
 	(label "SIDE_3"
 		(at 74.93 60.96 180)
+		(fields_autoplaced yes)
 		(effects
 			(font
@@
 	(label "SPARE_5"
 		(at 220.98 36.83 0)
+		(fields_autoplaced yes)
 		(effects
 			(font
@@
 	(label "SPARE_4a"
 		(at 21.59 66.04 0)
+		(fields_autoplaced yes)
 		(effects
 			(font
@@
 	(label "SIDE_6"
 		(at 74.93 45.72 180)
-		(effects
-			(font
+		(fields_autoplaced yes)
+		(effects
+			(font

Commit message: Firmware, and capacitor
Added firmware folder, and added additional capacitor in parallel to C15 in schematic. Footprint still needs to be added
Parts:
- removed TP2, TP3: TestPoint, TestPoint:TestPoint_Pad_2.0x2.0mm, symbol Connector:TestPoint
- added C16: 1uF, Capacitor_SMD:C_0603_1608Metric_Pad1.08x0.95mm_HandSolder, symbol Device:C
- renumbered C2 to C1, C11 to C10, C12 to C11, C13 to C12, C14 to C13, C15 to C14, C1 to C15, C3 to C2, C4 to C3, C5 to C4, C6 to C5, C7 to C6, C8 to C7, C9 to C8, C10 to C9
Connections:
- net GND: now also C16.2
- net UPDI: now also TP1.1; no longer J1.4 (Pin_4), J3.4 (Pin_4), J5.4 (Pin_4)
- net VCC: now also C16.1; no longer TP1.1
- net at D6.1 (DOUT): no longer D7.3 (DIN)
- net at D10.1 (DOUT): no longer D11.3 (DIN)
- net RX_J2: now reaches U2.11 (PB5)
- net RX_J2: now also J2.4 (Pin_4)
- net LED_J2-J5: now reaches U2.12 (PB4)
- net LED_J2-J5: now also D1.3 (DIN)
- net TX_J3: now reaches U2.13 (PB3)
- net TX_J3: now also J3.2 (Pin_2)
- net DATA_J4: now reaches U2.17 (PC0)
- net DATA_J4: now also J4.3 (Pin_3)
- net RX_J4: now reaches U2.18 (PC1)
- net RX_J4: now also J4.4 (Pin_4)
- net LED renamed LED_J1-J6
- net LED_J1-J6: now also D11.3 (DIN); no longer D1.3 (DIN)
- net LED_OUT_1: no longer names the net of D10.3 (DIN), D9.1 (DOUT)
- net SIDE_1 renamed DATA_J1
- net SIDE_2 renamed DATA_J2
- net DATA_J2: now also U2.10 (PB6); no longer U2.14 (PB2)
- net SIDE_3 renamed DATA_J3
- net DATA_J3: now also U2.14 (PB2); no longer U2.15 (PB1)
- net SIDE_4 renamed TX_J4
- net TX_J4: now also J4.2 (Pin_2); no longer J4.3 (Pin_3)
- net SIDE_5 renamed DATA_J5
- net DATA_J5: now also U2.21 (PC4); no longer U2.2 (PA3)
- net SIDE_6 renamed DATA_J6
- net DATA_J6: now also U2.1 (PA2); no longer U2.5 (PA4)
- net SPARE_1 renamed RX_J1
- net RX_J1: now also J1.4 (Pin_4); no longer J1.2 (Pin_2)
- net SPARE_2a renamed TX_J2
- removed net SPARE_2b: J2.4 (Pin_4), U2.10 (PB6)
- net SPARE_3 renamed LED_J3-J4
- net LED_J3-J4: now also D7.3 (DIN); no longer J3.2 (Pin_2)
- net SPARE_4a renamed TX_J5
- net TX_J5: now also J5.2 (Pin_2); no longer J4.2 (Pin_2)
- removed net SPARE_4b: J4.4 (Pin_4), U2.21 (PC4)
- net SPARE_5 renamed RX_J5
- net RX_J5: now also J5.4 (Pin_4); no longer J5.2 (Pin_2)
- net SPARE_6a renamed TX_J6
- net SPARE_6b renamed RX_J6
- net RX_J6: now also U2.2 (PA3); no longer U2.1 (PA2)
- new net RX_J3: J3.4 (Pin_4), U2.15 (PB1)
- new net TX_J1: J1.2 (Pin_2), U2.5 (PA4)
- no-connect marks 0 -> 3
Other:
- title: (none) -> PCB Tile Game
- moved on the sheet: C10, C11, C12, C13, C14, C15, C7, C8, C9, D10, D11, D12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
