File: Electrical Design/pcb_tile_game_tile_aaa/pcb_tile_game_tile_aaa.kicad_pcb (KiCad board)
At the start: 2 copper layers, 69.3 x 60 mm, 36 parts, among them J1 Conn_01x05_Pin, J2 Conn_01x05_Socket, J3 Conn_01x05_Pin, J4 Conn_01x05_Socket, J5 Conn_01x05_Pin, J6 Conn_01x05_Socket, U2 ATtiny3217-M

Commit message: created gerbers
Parts:
- moved G*** 1.33 mm to (137.6, 81.5)
Changed lines of the file:
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@@
 	(footprint "New Logo:byteSizedEngineeringLogo-6mm"
 		(layer "F.Cu")
-		(at 138.86 81.8)
+		(at 137.56 81.5)
 		(property "Reference" "G***"
 			(at 0 0 30)
@@
 		(fp_arc
 			(start 1.699999 -0.990938)
-			(mid 1.712519 -1.102166)
+			(mid 1.712521 -1.102165)
 			(end 1.749484 -1.207816)
 			(stroke
@@
 		(fp_arc
 			(start 1.046711 -1.856395)
-			(mid 1.638074 -1.79213)
+			(mid 1.63807 -1.792132)
 			(end 1.749484 -1.207815)
 			(stroke
@@
 		(fp_arc
 			(start 1.046711 -1.856395)
-			(mid 0.925123 -1.805473)
+			(mid 0.925123 -1.805472)
 			(end 0.794452 -1.788096)
 			(stroke
@@
 		(fp_arc
 			(start 1.04671 -1.856396)
-			(mid 0.925123 -1.805472)
+			(mid 0.925123 -1.805471)
 			(end 0.794452 -1.788094)
 			(stroke
@@
 		(fp_arc
 			(start -1.046711 1.280203)
-			(mid -1.638071 1.215938)
+			(mid -1.638072 1.215938)
 			(end -1.749484 0.631623)
 			(stroke
@@
 		(fp_arc
 			(start 1.046711 -1.856395)
-			(mid 1.638074 -1.79213)
+			(mid 1.63807 -1.792132)
 			(end 1.749484 -1.207815)
 			(stroke
@@
 		(fp_arc
 			(start 1.046711 -1.856395)
-			(mid 1.63807 -1.792132)
+			(mid 1.638074 -1.79213)
 			(end 1.749484 -1.207815)
 			(stroke
@@
 		(fp_arc
 			(start 1.046711 -1.856395)
-			(mid 0.925123 -1.805472)
+			(mid 0.925123 -1.805473)
 			(end 0.794453 -1.788096)
 			(stroke
@@
 		(fp_arc
 			(start 0.794452 1.211902)
-			(mid 0.925123 1.22928)
+			(mid 0.925123 1.229281)
 			(end 1.046712 1.280202)
 			(stroke
@@
 		(fp_arc
 			(start 1.046711 -1.856395)
-			(mid 1.638074 -1.79213)
+			(mid 1.63807 -1.792132)
 			(end 1.749484 -1.207815)
 			(stroke
@@
 		(fp_arc
 			(start -1.046711 1.280203)
-			(mid -1.638071 1.215938)
+			(mid -1.638072 1.215938)
 			(end -1.749484 0.631623)
 			(stroke
@@
 		(fp_arc
 			(start 1.046711 -1.856395)
-			(mid 0.925123 -1.805471)
+			(mid 0.925124 -1.805471)
 			(end 0.794452 -1.788097)
 			(stroke
@@
 		(fp_arc
 			(start 1.046711 -1.856395)
-			(mid 1.638074 -1.79213)
+			(mid 1.63807 -1.792132)
 			(end 1.749484 -1.207815)
 			(stroke
@@
 		(fp_arc
 			(start 1.699999 -0.990938)
-			(mid 1.712519 -1.102166)
+			(mid 1.712521 -1.102165)
 			(end 1.749484 -1.207816)
 			(stroke
@@
 		(fp_arc
 			(start 1.046711 -1.856395)
-			(mid 1.638074 -1.79213)
+			(mid 1.63807 -1.792132)
 			(end 1.749484 -1.207815)
 			(stroke
@@
 		(fp_arc
 			(start 1.046711 -1.856395)
-			(mid 0.925123 -1.805473)
+			(mid 0.925123 -1.805472)
 			(end 0.794452 -1.788096)
 			(stroke
@@
 		(fp_arc
 			(start 1.046711 -1.856395)
-			(mid 1.638074 -1.79213)
+			(mid 1.63807 -1.792132)
 			(end 1.749484 -1.207815)
 			(stroke
@@
 		(fp_arc
 			(start -1.046711 1.280203)
-			(mid -1.638071 1.215938)
+			(mid -1.638072 1.215938)
 			(end -1.749484 0.631623)
 			(stroke
@@
 		(fp_arc
 			(start 1.699999 -0.990938)
-			(mid 1.712519 -1.102166)
+			(mid 1.712521 -1.102165)
 			(end 1.749484 -1.207816)
 			(stroke
@@
 		(fp_arc
 			(start 1.046711 -1.856395)
-			(mid 1.638074 -1.79213)
+			(mid 1.63807 -1.792132)
 			(end 1.749484 -1.207815)
 			(stroke
@@
 		(fp_arc
 			(start 1.046711 -1.856395)
-			(mid 0.925123 -1.805473)
+			(mid 0.925123 -1.805472)
 			(end 0.794452 -1.788096)
 			(stroke
@@
 	)
 	(gr_text "Rev ${REVISION}"
-		(at 147.16 84.7 0)
+		(at 146.56 81.5 0)
 		(layer "F.SilkS")
 		(effects
@@
 	)
 	(gr_text "${TITLE}"
-		(at 147.16 77.2 0)
+		(at 146.56 77.2 0)
 		(layer "F.SilkS")
 		(effects
@@
 		)
 	)
-	(group ""
-		(members "2ce42902-ce35-42dd-82a2-fd03e3ee6900" "d9f889fc-7e00-493b-8d3f-5fbc6097f20e")
-	)
 )
