File: Electrical Design/pcb_tile_game_tile_ooo/pcb_tile_game_tile_ooo.kicad_pcb (KiCad board)
At the start: 2 copper layers, 69.3 x 60 mm, 44 parts, among them J1 Conn_01x05_Pin, J2 Conn_01x05_Socket, J3 Conn_01x05_Pin, J4 Conn_01x05_Socket, J5 Conn_01x05_Pin, J6 Conn_01x05_Socket, U2 ATtiny3217-M

Commit message: created gerbers
Parts:
- moved G*** 27.1 mm to (128.1, 104.5)
Changed lines of the file:
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@@
 			(drillshape 0)
 			(scaleselection 1)
-			(outputdirectory "")
+			(outputdirectory "ooo.gerbers")
 		)
 	)
@@
 	(footprint "New Logo:byteSizedEngineeringLogo-6mm"
 		(layer "F.Cu")
-		(at 115.76 80.4)
+		(at 128.06 104.5)
 		(property "Reference" "G***"
 			(at 0 0 30)
@@
 	)
 	(gr_text "Rev ${REVISION}"
-		(at 165.86 81.4 0)
+		(at 150.321904 105.5 0)
 		(layer "F.SilkS")
 		(effects
 			(font
-				(size 2 2)
-				(thickness 0.4)
+				(size 1 1)
+				(thickness 0.2)
 				(bold yes)
 			)
@@
 	)
 	(gr_text "${TITLE}"
-		(at 140.06 72.1 0)
+		(at 153.06 103.5 0)
 		(layer "F.SilkS")
 		(effects
 			(font
-				(size 2 2)
-				(thickness 0.4)
+				(size 1 1)
+				(thickness 0.2)
 				(bold yes)
 			)
