File: Electrical Design/pcb_tile_game_tile_ooo/pcb_tile_game_tile_ooo.kicad_sch (KiCad schematic)
At the start: 43 parts, among them J1 Conn_01x05_Pin, J2 Conn_01x05_Socket, J3 Conn_01x05_Pin, J4 Conn_01x05_Socket, J5 Conn_01x05_Pin, J6 Conn_01x05_Socket, U2 ATtiny3217-M

Commit message: created gerbers
Connections:
- net LED_J1-J4 renamed LED_J4-J1
- net LED_J2-J5 renamed LED_J5-J2
- net LED_J3-J6 renamed LED_J6-J3
Changed lines of the file:
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@@
 	(label "RX_J1"
 		(at 140.97 31.75 0)
-		(fields_autoplaced yes)
 		(effects
 			(font
@@
 	(label "TX_J5"
 		(at 21.59 66.04 0)
-		(fields_autoplaced yes)
 		(effects
 			(font
@@
 	(label "RX_J3"
 		(at 74.93 60.96 180)
-		(fields_autoplaced yes)
 		(effects
 			(font
@@
 	(label "DATA_J4"
 		(at 21.59 58.42 0)
-		(fields_autoplaced yes)
 		(effects
 			(font
@@
 	(label "TX_J1"
 		(at 74.93 45.72 180)
-		(fields_autoplaced yes)
 		(effects
 			(font
@@
 	(label "UPDI"
 		(at 74.93 35.56 180)
-		(fields_autoplaced yes)
 		(effects
 			(font
@@
 	(label "RX_J6"
 		(at 74.93 43.18 180)
-		(fields_autoplaced yes)
 		(effects
 			(font
@@
 	(label "DATA_J5"
 		(at 220.98 34.29 0)
-		(fields_autoplaced yes)
-		(effects
-			(font
-				(size 1.27 1.27)
-			)
-			(justify left bottom)
-		)
-	)
-	(label "LED_J1-J4"
+		(effects
+			(font
+				(size 1.27 1.27)
+			)
+			(justify left bottom)
+		)
+	)
+	(label "LED_J4-J1"
 		(at 21.59 140.97 0)
-		(fields_autoplaced yes)
 		(effects
 			(font
@@
 	(label "TX_J6"
 		(at 74.93 38.1 180)
-		(fields_autoplaced yes)
 		(effects
 			(font
@@
 	(label "DATA_J5"
 		(at 21.59 68.58 0)
-		(fields_autoplaced yes)
 		(effects
 			(font
@@
 	(label "RX_J6"
 		(at 220.98 60.96 0)
-		(fields_autoplaced yes)
 		(effects
 			(font
@@
 	(label "RX_J5"
 		(at 21.59 71.12 0)
-		(fields_autoplaced yes)
 		(effects
 			(font
@@
 	(label "DATA_J1"
 		(at 74.93 48.26 180)
-		(fields_autoplaced yes)
-		(effects
-			(font
-				(size 1.27 1.27)
-			)
-			(justify right bottom)
-		)
-	)
-	(label "LED_J3-J6"
+		(effects
+			(font
+				(size 1.27 1.27)
+			)
+			(justify right bottom)
+		)
+	)
+	(label "LED_J6-J3"
 		(at 74.93 53.34 180)
-		(fields_autoplaced yes)
 		(effects
 			(font
@@
 	(label "DATA_J2"
 		(at 74.93 73.66 180)
-		(fields_autoplaced yes)
 		(effects
 			(font
@@
 	(label "UPDI"
 		(at 88.9 41.91 180)
-		(fields_autoplaced yes)
 		(effects
 			(font
@@
 	(label "DATA_J3"
 		(at 180.34 34.29 0)
-		(fields_autoplaced yes)
 		(effects
 			(font
@@
 	(label "DATA_J4"
 		(at 180.34 58.42 0)
-		(fields_autoplaced yes)
 		(effects
 			(font
@@
 	(label "RX_J4"
 		(at 21.59 60.96 0)
-		(fields_autoplaced yes)
 		(effects
 			(font
@@
 	(label "DATA_J1"
 		(at 140.97 34.29 0)
-		(fields_autoplaced yes)
 		(effects
 			(font
@@
 	(label "RX_J2"
 		(at 140.97 60.96 0)
-		(fields_autoplaced yes)
-		(effects
-			(font
-				(size 1.27 1.27)
-			)
-			(justify left bottom)
-		)
-	)
-	(label "LED_J3-J6"
+		(effects
+			(font
+				(size 1.27 1.27)
+			)
+			(justify left bottom)
+		)
+	)
+	(label "LED_J6-J3"
 		(at 22.86 170.18 0)
-		(fields_autoplaced yes)
 		(effects
 			(font
@@
 	(label "DATA_J2"
 		(at 140.97 58.42 0)
-		(fields_autoplaced yes)
-		(effects
-			(font
-				(size 1.27 1.27)
-			)
-			(justify left bottom)
-		)
-	)
-	(label "LED_J2-J5"
+		(effects
+			(font
+				(size 1.27 1.27)
+			)
+			(justify left bottom)
+		)
+	)
+	(label "LED_J5-J2"
 		(at 21.59 63.5 0)
-		(fields_autoplaced yes)
 		(effects
 			(font
@@
 	(label "RX_J4"
 		(at 180.34 60.96 0)
-		(fields_autoplaced yes)
 		(effects
 			(font
@@
 	(label "DATA_J6"
 		(at 220.98 58.42 0)
-		(fields_autoplaced yes)
 		(effects
 			(font
@@
 	(label "RX_J2"
 		(at 74.93 71.12 180)
-		(fields_autoplaced yes)
-		(effects
-			(font
-				(size 1.27 1.27)
-			)
-			(justify right bottom)
-		)
-	)
-	(label "LED_J2-J5"
+		(effects
+			(font
+				(size 1.27 1.27)
+			)
+			(justify right bottom)
+		)
+	)
+	(label "LED_J5-J2"
 		(at 21.59 111.76 0)
-		(fields_autoplaced yes)
 		(effects
 			(font
@@
 	(label "TX_J1"
 		(at 140.97 36.83 0)
-		(fields_autoplaced yes)
 		(effects
 			(font
@@
 	(label "TX_J4"
 		(at 180.34 55.88 0)
-		(fields_autoplaced yes)
 		(effects
 			(font
@@
 	(label "TX_J3"
 		(at 180.34 36.83 0)
-		(fields_autoplaced yes)
 		(effects
 			(font
@@
 	(label "RX_J3"
 		(at 180.34 31.75 0)
-		(fields_autoplaced yes)
 		(effects
 			(font
@@
 	(label "TX_J2"
 		(at 140.97 55.88 0)
-		(fields_autoplaced yes)
 		(effects
 			(font
@@
 	(label "RX_J1"
 		(at 74.93 50.8 180)
-		(fields_autoplaced yes)
-		(effects
-			(font
-				(size 1.27 1.27)
-			)
-			(justify right bottom)
-		)
-	)
-	(label "LED_J1-J4"
+		(effects
+			(font
+				(size 1.27 1.27)
+			)
+			(justify right bottom)
+		)
+	)
+	(label "LED_J4-J1"
 		(at 74.93 68.58 180)
-		(fields_autoplaced yes)
 		(effects
 			(font
@@
 	(label "TX_J2"
 		(at 74.93 76.2 180)
-		(fields_autoplaced yes)
 		(effects
 			(font
@@
 	(label "TX_J6"
 		(at 220.98 55.88 0)
-		(fields_autoplaced yes)
 		(effects
 			(font
@@
 	(label "TX_J3"
 		(at 74.93 66.04 180)
-		(fields_autoplaced yes)
 		(effects
 			(font
@@
 	(label "UPDI"
 		(at 100.33 27.94 0)
-		(fields_autoplaced yes)
 		(effects
 			(font
@@
 	(label "DATA_J3"
 		(at 74.93 63.5 180)
-		(fields_autoplaced yes)
 		(effects
 			(font
@@
 	(label "TX_J5"
 		(at 220.98 36.83 0)
-		(fields_autoplaced yes)
 		(effects
 			(font
@@
 	(label "TX_J4"
 		(at 74.93 58.42 180)
-		(fields_autoplaced yes)
 		(effects
 			(font
@@
 	(label "RX_J5"
 		(at 220.98 31.75 0)
-		(fields_autoplaced yes)
 		(effects
 			(font
@@
 	(label "DATA_J6"
 		(at 74.93 40.64 180)
-		(fields_autoplaced yes)
-		(effects
-			(font
+		(effects
+			(font
