File: Electrical Design/pcb_tile_game_tile_sos/pcb_tile_game_tile_sos.kicad_pcb (KiCad board)
At the start: 2 copper layers, 69.3 x 60 mm, 40 parts, among them J1 Conn_01x05_Pin, J2 Conn_01x05_Socket, J3 Conn_01x05_Pin, J4 Conn_01x05_Socket, J5 Conn_01x05_Pin, J6 Conn_01x05_Socket, U2 ATtiny3217-M

Commit message: created gerbers
Routing:
- net /TX_J6: track 15.8 -> 24.0 mm
- net /UPDI: track 28.2 -> 30.4 mm
- net /TX_J5: track 36.5 -> 35.0 mm
- net /RX_J5: track 33.4 -> 31.9 mm
- net /DATA_J5: track 34.9 -> 33.5 mm
