File: Electrical Design/pcb_tile_game_tile_ssa/pcb_tile_game_tile_ssa.kicad_pcb (KiCad board)
At the start: 2 copper layers, 69.3 x 60 mm, 38 parts, among them J1 Conn_01x05_Pin, J2 Conn_01x05_Socket, J3 Conn_01x05_Pin, J4 Conn_01x05_Socket, J5 Conn_01x05_Pin, J6 Conn_01x05_Socket, U2 ATtiny3217-M

Commit message: created gerbers
Changed lines of the file:
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@@
 			(drillshape 0)
 			(scaleselection 1)
-			(outputdirectory "")
+			(outputdirectory "ssa.gerbers")
 		)
 	)
@@
 		(fp_arc
 			(start 1.699999 -0.990938)
-			(mid 1.712522 -1.102165)
+			(mid 1.712523 -1.102165)
 			(end 1.749485 -1.207816)
 			(stroke
@@
 		(fp_arc
 			(start 1.749484 0.631624)
-			(mid 1.71251 0.525976)
+			(mid 1.712509 0.525977)
 			(end 1.699999 0.414747)
 			(stroke
@@
 		(fp_arc
 			(start 1.699999 -0.990938)
-			(mid 1.712522 -1.102165)
+			(mid 1.712523 -1.102165)
 			(end 1.749485 -1.207816)
 			(stroke
@@
 		(fp_arc
 			(start -1.749485 -1.207816)
-			(mid -1.712522 -1.102165)
+			(mid -1.71252 -1.102166)
 			(end -1.699999 -0.990938)
 			(stroke
@@
 		(fp_arc
 			(start 1.699999 -0.990938)
-			(mid 1.712522 -1.102165)
+			(mid 1.712523 -1.102165)
 			(end 1.749485 -1.207816)
 			(stroke
